Commit message: Modified package

File: pxpincher_description/urdf/pincher_gripper.xacro (robot description, xacro)
@@ -25,5 +25,5 @@
       <origin xyz="0 0 0" rpy="0 0 0"/>
       <axis xyz="1 0 0"/>
-      <limit effort="30" velocity="0.5" lower="-1" upper="1"/>
+      <limit effort="30" velocity="0.5" lower="-0.01" upper="0.0"/>
       <parent link="gripper_servo_link"/>
       <child link="gripper_active_link"/>
@@ -57,8 +57,16 @@
       <origin xyz="0 0 0" rpy="0 0 0"/>
       <axis xyz="1 0 0"/>
-      <limit effort="30" velocity="0.5" lower="-10" upper="10"/>
+      <limit effort="30" velocity="0.5" lower="0.0" upper="0.02"/>
       <parent link="gripper_servo_link"/>
       <child link="gripper_active2_link"/>
       <mimic joint="gripper_joint" multiplier="-${FACTOR_GRIPPER_TRANSL}"  offset = "-${OFFSET_GRIPPER_TRANSL}"/>
     </joint>
+<!-- Edit Strats 30-11-2015 -->
+ <gazebo reference="gripper_active_link">
+     <gravity>false</gravity>
+ </gazebo>
+ <gazebo reference="gripper_active2_link">
+     <gravity>false</gravity>
+ </gazebo>
+<!-- Edit Ends 30-11-2015 -->
 </robot>
