Commit message: Update pincher_arm.urdf.xacro

File: pxpincher_description/urdf/pincher_arm.urdf.xacro (robot description, xacro)
@@ -4,6 +4,5 @@
     <!-- We can configure joints velocity limit and lower/upper limits
           to allow access to different operational areas, e.g. left handed vs. right handed robot -->
-<!-- Edit Starts  -->
- <xacro:property name="joints_vlimit" value="1.571"/>
+   <xacro:property name="joints_vlimit" value="1.571"/>
     <xacro:property name="pan_llimit" value="-1.17"/>
     <xacro:property name="pan_ulimit" value="1.43"/>
@@ -17,8 +16,8 @@
      <!-- Pincher arm is same as Turtlebot -->
     <xacro:include filename="$(find pxpincher_description)/urdf/turtlebot_arm.xacro"/>
-    <!-- As we don't have here a turtlebot base, add a base_link1 link as its location reference -->
-    <link name="base_link1"/>
+    <!-- As we don't have here a turtlebot base, add a base_link link as its location reference -->
+    <link name="base_link"/>
     <!-- Turtlebot arm macro -->
-    <turtlebot_arm parent="base_link1" color="Gray" gripper_color="Gray"   pincher_gripper="true" turtlebot_gripper="false">
+    <turtlebot_arm parent="base_link" color="Gray" gripper_color="Gray"   pincher_gripper="true" turtlebot_gripper="false">
       <!-- Place the "floating" arm at the location it should be if mounted on a turtlebot,
            as pick and place and other demos assume this location -->
@@ -41,4 +40,3 @@
 </visual>
 </link>
-<!-- Edit ends -->
 </robot>

Commit message: Renamend arm_controller_link to arm_mount_link (I cannot change arm_base_link to the new mount-plate, since it would break compatibility with existing code). I also moved the origin of the mount-plate to a new location

File: pxpincher_description/urdf/pincher_arm.urdf.xacro (robot description, xacro)
@@ -24,19 +24,21 @@
       <origin xyz="0.06 0 0.01"/>
     </turtlebot_arm>
-<!-- Phantomx Arm Controller link-->
-<joint name="arm_controller_joint" type="fixed">
-      <origin xyz="-0.09 -0.06 -0.105" rpy="0 0 0"/>
-      <parent link="arm_base_link"/>
-      <child link="arm_controller_link"/>
-      <axis xyz="0 0 1"/>
+<!-- Phantomx Arm mount/Controllerboard link-->
+<joint name="arm_mount_joint" type="fixed">
+   <!--origin xyz="-0.09 -0.06 -0.105" rpy="0 0 0"/-->
+   <origin xyz="0.025 0.0 -0.06" rpy="0 0 0"/>
+   <parent link="arm_base_link"/>
+   <child link="arm_mount_link"/>
+   <axis xyz="0 0 1"/>
  </joint>
-<link name="arm_controller_link">
+<link name="arm_mount_link">
  <visual>
-<origin xyz="0.18 -0.01 0.05" rpy="0 0 7.85"/>
-<geometry>
- <mesh filename="package://pxpincher_description/meshes/arm_controller_link.stl" scale="0.007 0.007 0.007"/>
- </geometry>
- <material name="Gray"/>
-</visual>
+   <!--origin xyz="0.18 -0.01 0.05" rpy="0 0 7.85"/-->
+   <origin xyz="0.0825 -0.09 0.0" rpy="0 0 1.57"/>
+   <geometry>
+     <mesh filename="package://pxpincher_description/meshes/arm_mount.stl" scale="0.009 0.009 0.009"/>
+    </geometry>
+   <material name="Gray"/>
+  </visual>
 </link>
 </robot>

Commit message: Size of the robot base corrected according to the real one

File: pxpincher_description/urdf/pincher_arm.urdf.xacro (robot description, xacro)
@@ -27,5 +27,5 @@
 <joint name="arm_mount_joint" type="fixed">
    <!--origin xyz="-0.09 -0.06 -0.105" rpy="0 0 0"/-->
-   <origin xyz="0.025 0.0 -0.06" rpy="0 0 0"/>
+   <origin xyz="0.04 0.0 -0.065" rpy="0 0 0"/>
    <parent link="arm_base_link"/>
    <child link="arm_mount_link"/>
@@ -35,7 +35,7 @@
  <visual>
    <!--origin xyz="0.18 -0.01 0.05" rpy="0 0 7.85"/-->
-   <origin xyz="0.0825 -0.09 0.0" rpy="0 0 1.57"/>
+   <origin xyz="0.091 -0.1 0.0" rpy="0 0 1.57"/>
    <geometry>
-     <mesh filename="package://pxpincher_description/meshes/arm_mount.stl" scale="0.009 0.009 0.009"/>
+     <mesh filename="package://pxpincher_description/meshes/arm_mount.stl" scale="0.01 0.01 0.01"/>
     </geometry>
    <material name="Gray"/>
